Commit message: sim: drive head pitch from /mars/head/set_position
The webapp's head-tilt slider publishes /mars/head/set_position (degrees) and
reads back /mars/head/current_position, but the sim never wired either up, so
the slider sat disabled at "-" and the head never moved.

Mirror the arm path: the bridge subscribes to set_position and enqueues a
HeadCmd, the sim node drives the joint_head DOF (immediate, clamped), and the
sim node + bridge republish current_position (with limits) so the slider
self-calibrates. The head camera chain is fixed-jointed to the head link, so
the view tilts for free. Range is +/-20 deg; the URDF joint_head limit is set
to match so the full range is reachable. Head is not gated by arm torque,
matching the real robot.

Co-Authored-By: Claude Opus 4.8 (1M context) <noreply@anthropic.com>

File: ros2_ws/src/mars_bot/mars_sim/urdf/mars.urdf (robot description, URDF)
Before this commit: robot mars_bot, 17 links, 16 joints
Joints:
- joint joint_head: limit lower=-0.1745 upper=0.5236 effort=2.0 velocity=2.0 -> lower=-0.3491 upper=0.3491 effort=2.0 velocity=2.0

Commit message: feat(sim): replace the Genesis sim with a MuJoCo digital-twin driver
The sim no longer runs its own robot approximation behind a WebSocket
bridge: mars_sim_driver is a new ROS 2 package that impersonates the
hardware drivers at the topic level -- same topics, types, rates, frames
(odom/TF @30Hz, /scan @6Hz, cameras @7.5/5Hz, depth+points @8Hz with the
real stereo's [0.25,2]m clamp) -- so Nav2, AMCL, the brain, and the webapp
run unmodified. Three layers, each usable without the ones above: world.py
(pure MJCF+URDF model building, the future GPU-backend seam), core.py
(VirtualMars -- the whole simulated robot as one importable, zero-ROS
object), node.py (the ROS wrapper; physics on a steady clock, renders on a
separate thread, lazy camera topics). grid_localizer_sim stands in for the
CUDA-only localizer with the identical lifecycle + service contract.

The real navigation stack replaces the genesis-era special cases:
navigate_to_position_sim and the catalog swap machinery are deleted -- the
sim runs the robot's own navigate_to_position against the real
bt_navigator/MPPI/AMCL. Collision geometry is the res-200 CoACD bake (1301
hulls, stress-gated: 3 tour loops, no divergence, max 2.79 m/s). goto_js*
inputs are shape-validated and the physics thread survives faults.

Co-Authored-By: Claude Fable 5 <noreply@anthropic.com>

File: ros2_ws/src/mars_bot/mars_sim/urdf/mars.urdf (robot description, URDF)
Before this commit: robot mars_bot, 17 links, 16 joints
Joints:
- joint joint6: limit lower=-0.8727 upper=0.3491 effort=2.0 velocity=2.0 -> lower=0 upper=0.8727 effort=2.0 velocity=2.0
- joint joint6M: limit lower=-0.8727 upper=0.3491 effort=2.0 velocity=2.0 -> lower=-0.8727 upper=0 effort=2.0 velocity=2.0
