Commit message: Revert "webapp, sim, and WebRTC: per-client protocol, agent/skills surfaces, brain state broadcasts"

File: ros2_ws/src/mars_bot/mars_sim/urdf/mars.urdf (robot description, URDF)
Before this commit: robot mars_bot, 17 links, 16 joints
Joints:
- joint joint_head: limit lower=-0.3491 upper=0.3491 effort=2.0 velocity=2.0 -> lower=-0.1745 upper=0.5236 effort=2.0 velocity=2.0

Commit message: feat(sim): gripper contact model, precise robot collisions, props, and pick-anything fidelity
The gripper couldn't grip: each finger blade was one bounding slab that
held the closed fingertips 2.4mm apart everywhere. The blades are now a
pivot pin plus 4 min-area boxes along the hook with a single-box grip pad
(a segmented pad is serrated and rolls cans and balls straight out), the
gripper servo runs on joint6's real 2 N*m rating instead of the 50 N*m
arm clamp, and finger damping lives on the joint where implicitfast
integrates it stably. base_link grows from one box to 8 primitives
(rear tray, wheels, arm mount, lidar turret, neck), link1-3 get 3 each.
MuJoCo-only contact settings live in world.tune_contacts; the drive
wheels are frictionless (condim 1 + priority) because the z-pinned planar
base otherwise answers every step with ~50N of spurious normal force
whose friction cone pins the robot.

Five graspable props (cube, can, sock, bar, ball) park off-map until
core.drop_objects lays them out in front of the robot; each is shaped by
what pick_any_object's pipeline needs -- sizes inside the 81mm jaw, tops
inside the skill's closing band, colours that don't starve the LK flow
tracker, the ball foam-soft because a hard sphere's contact rolls around
the curve and the arm rides up over it.

Running the SHIPPED pick_any_object skill exposed each place the sim
diverged from the robot it was tuned on; all fixes are sim-side:
cameras at the real drivers' rates (10/6 Hz), the head camera at the
real lens's focal length (fx ~= 355, back-solved from the skill's own
tuning notes; wrist keeps 80 deg until measured), the arm sags past its
encoders (~19mm at the pick pose) with /joint_states reporting
encoder-side angles like the machine, gotos complete on ARRIVAL inside
manipulation_server's time+0.2s budget, and the stopped base holds
station instead of letting the arm's reaction torque walk it mid-grasp.

Shipped skill, clean starts: cube 4/4, bar 6/6, can 6/6, sock 5/6,
ball 4/6; wave and the arm skills unaffected.

File: ros2_ws/src/mars_bot/mars_sim/urdf/mars.urdf (robot description, URDF)
Before this commit: robot mars_bot, 17 links, 16 joints
Links:
- link base_link: geometry collision box size=0.0374 0.036 0.0366; collision box size=0.051 0.0854 0.039
- link link1: geometry collision box size=0.0403 0.0226 0.0466; collision box size=0.0465 0.04 0.0216
- link link2: geometry collision box size=0.0244 0.0475 0.0436; collision box size=0.035 0.054 0.0763
- link link3: geometry collision box size=0.028 0.0467 0.031; collision box size=0.0677 0.054 0.035
- link link61: geometry collision box size=0.0022 0.0045 0.0389; collision box size=0.0022 0.0062 0.0389
- link link62: geometry collision box size=0.0022 0.0045 0.0389; collision box size=0.0022 0.0062 0.0389
